Commit message: fixed arm, controller still not reliable

File: urdf/arm/arm.urdf.xacro (robot description, xacro)
@@ -3,130 +3,157 @@
   <xacro:macro name="simple_arm" params="parent_link *origin">
   <xacro:include filename="$(find irobot_create_description)/urdf/common_properties.urdf.xacro"/>
-  <joint name="arm_base_joint" type="fixed">
+  <xacro:property name="mass" value="0.00001" />
+  <xacro:property name="link_len" value="0.25" />
+  <xacro:property name="wrist_len" value="0.05" />
+  <xacro:property name="effort_max" value="1000" />
+  <xacro:property name="velocity_max" value="10" />
+  <xacro:property name="inertial_elem" value="0.001" />
+  <joint name="robot_to_base" type="fixed">
+    <xacro:insert_block name="origin"/>
     <parent link="${parent_link}"/>
     <child link="arm_base_link"/>
-    <xacro:insert_block name="origin"/>
   </joint>
-  <link name="arm_rgbd_camera_frame">
-    <xacro:inertial_dummy/>
-  </link>
   <link name='arm_base_link'>
-      <xacro:inertial_cylinder mass="0.17" radius="0.1" length="0.1"/>
-      <collision name="arm_base_link_collision">
-        <pose>0 0 0 0 0 0</pose>
+    <inertial>
+      <mass value="${mass}"/>
+      <inertia ixx="${inertial_elem}" ixy="0.0" ixz="0.0" iyy="${inertial_elem}" iyz="0.0" izz="${inertial_elem}"/>
+    </inertial>
+      <visual name='arm_base_link_visual'>
+        <origin xyz="0 0 0"/>
         <geometry>
-          <cylinder radius="0.1" length="0.1"/>
+          <cylinder radius="0.05" length="0.001"/>
         </geometry>
-      </collision>
-      <visual name='arm_base_link_visual'>
-        <pose>0 0 0 0 0 0</pose>
-        <geometry>
-          <cylinder radius="0.1" length="0.1"/>
-        </geometry>
-        <material name="black">
-          <diffuse>0.05 0.05 0.05</diffuse>
-        </material>
+      <material name="grey">
+        <color rgba="0.2 0.2 0.2 1"/>
+      </material>
       </visual>
     </link>
-    <link name='lower_arm_link'>
-      <pose relative_to='arm_base_link'>0.375 0.0 0.0 0 1.570796 0</pose>
-      <xacro:inertial_cylinder mass="0.17" radius="0.1" length="0.75"/>
-      <collision name='lower_link_collision'>
+  <joint name="arm_base_joint" type="continuous">
+    <axis xyz="0 0 1"/>
+    <origin xyz="0.0 0 0.002" rpy="0 0 0"/>
+    <parent link="arm_base_link"/>
+    <child link="arm_base2_link"/>
+    <limit effort="${effort_max}" velocity="${velocity_max}"/>
+  </joint>
+  <link name='arm_base2_link'>
+    <inertial>
+      <mass value="${mass}"/>
+      <inertia ixx="${inertial_elem}" ixy="0.0" ixz="0.0" iyy="${inertial_elem}" iyz="0.0" izz="${inertial_elem}"/>
+    </inertial>
+      <visual name='arm_base2_link'>
+        <origin xyz="0 0 0"/>
         <geometry>
-          <cylinder radius="0.1" length="0.5"/>
+          <cylinder radius="0.05" length="0.01"/>
         </geometry>
-      </collision>
+      <material name="grey">
+        <color rgba="0.2 0.2 0.2 1"/>
+      </material>
+      </visual>
+  </link>
+  <joint name="arm_shoulder_joint" type="continuous">
+    <axis xyz="0 1 0"/>
+    <origin xyz="0.0 0 0.01" rpy="0 0 0"/>
+    <parent link="arm_base2_link"/>
+    <child link="arm_shoulder_link"/>
+    <limit effort="${effort_max}" velocity="${velocity_max}"/>
+  </joint>
+<link name='arm_shoulder_link'>
+    <inertial>
+      <origin xyz="0 0 ${link_len/2}"/>
+      <mass value="${mass}"/>
+      <inertia ixx="${inertial_elem}" ixy="0.0" ixz="0.0" iyy="${inertial_elem}" iyz="0.0" izz="${inertial_elem}"/>
+    </inertial>
       <visual name='lower_link_visual'>
+        <origin xyz="0 0 ${link_len/2}"/>
         <geometry>
-          <cylinder radius="0.1" length="0.75"/>
+          <cylinder radius="0.01" length="${link_len}"/>
         </geometry>
-        <material name="black">
-          <diffuse>0.05 0.05 0.05</diffuse>
-        </material>
+      <material name="grey">
+        <color rgba="0.2 0.2 0.2 1"/>
+      </material>
       </visual>
-    </link>
-    <link name='upper_arm_link'>
-      <pose relative_to='joint_1'>0.375 0.0 0.0 0 1.570796 0</pose>
-      <xacro:inertial_cylinder mass="0.17" radius="0.1" length="0.75"/>
-      <collision name='upper_link_collision'>
+  </link>
+  <joint name="arm_elbow_joint" type="continuous">
+    <axis xyz="0 1 0"/>
+    <origin xyz="0.0 0 ${link_len}" rpy="0 0 0"/>
+    <parent link="arm_shoulder_link"/>
+    <child link="arm_elbow_link"/>
+    <limit effort="${effort_max}" velocity="${velocity_max}"/>
+  </joint>
+  <link name='arm_elbow_link'>
+    <inertial>
+      <origin xyz="0 0 ${link_len/2}"/>
+      <mass value="${mass}"/>
+      <inertia ixx="${inertial_elem}" ixy="0.0" ixz="0.0" iyy="${inertial_elem}" iyz="0.0" izz="${inertial_elem}"/>
+    </inertial>
+      <visual name='lower_link_visual'>
+        <origin xyz="0 0 ${link_len/2}"/>
         <geometry>
-          <cylinder radius="0.1" length="0.5"/>
+          <cylinder radius="0.01" length="${link_len}"/>
         </geometry>
-      </collision>
-      <visual name='upper_link_visual'>
+      <material name="grey">
+        <color rgba="0.2 0.2 0.2 1"/>
+      </material>
+      </visual>
+  </link>
+  <joint name="arm_wrist_joint" type="continuous">
+    <axis xyz="0 1 0"/>
+    <origin xyz="0.0 0 ${link_len}" rpy="0 0 0"/>
+    <parent link="arm_elbow_link"/>
+    <child link="arm_wrist_link"/>
+    <limit effort="${effort_max}" velocity="${velocity_max}"/>
+  </joint>
+  <link name='arm_wrist_link'>
+    <inertial>
+      <origin xyz="0 0 ${wrist_len/2}"/>
+      <mass value="${mass}"/>
+      <inertia ixx="${inertial_elem}" ixy="0.0" ixz="0.0" iyy="${inertial_elem}" iyz="0.0" izz="${inertial_elem}"/>
+    </inertial>
+      <visual name='lower_link_visual'>
+        <origin xyz="0 0 ${wrist_len/2}"/>
         <geometry>
-          <cylinder radius="0.1" length="0.75"/>
+          <cylinder radius="0.01" length="${wrist_len}"/>
         </geometry>
-        <material name="black">
-          <diffuse>0.05 0.05 0.05</diffuse>
-        </material>
+      <material name="grey">
+        <color rgba="0.2 0.2 0.2 1"/>
+      </material>
       </visual>
-    </link>
-    <frame name="gripper_mount_point">
-      <pose relative_to='joint_2'>0.0 0 0 0 0 0</pose>
-    </frame>
-    <include>
-      <name>gripper</name>
-      <uri>model://mbzirc_oberon7_gripper</uri>
-      <placement_frame>mount_point</placement_frame>
-      <pose relative_to="gripper_mount_point">0 0 0 0 0 0</pose>
-    </include>
-    <joint name='joint_0' type='revolute'>
-      <pose relative_to='arm_base_link'>0.0 0.0 0.0 0 0 0</pose>
-      <parent link="arm_base_link"/>
-      <child link="lower_arm_link"/>
-      <axis>
-        <xyz>0 -1 0</xyz>
-      </axis>
-      <limit effort="500" velocity="0.15" lower="-1.570796" upper="1.5707896"/>
+  </link>
+  <frame name="camera_mount_point">
+      <pose relative_to='arm_wrist_link'>0.0 0 0 0 0 0</pose>
+  </frame>
+  <ros2_control name="arm_controller_hw" type="system">
+    <hardware>
+      <plugin>ign_ros2_control/IgnitionSystem</plugin>
+    </hardware>
+    <joint name="arm_base_joint">
+      <command_interface name="position"/>
+      <state_interface name="position">
+        <param name="initial_value">0.0</param>
+      </state_interface>
+      <state_interface name="velocity"/>
     </joint>
-    <joint name='joint_1' type='revolute'>
-      <pose relative_to='joint_0'>0.75 0.0 0.0 0 1.570796 0</pose>
-      <parent link="lower_arm_link"/>
-      <child link="upper_arm_link"/>
-      <axis>
-        <xyz>0 -1 0</xyz>
-      </axis>
-      <limit effort="500" velocity="0.15" lower="-1.570796" upper="1.5707896"/>
+    <joint name="arm_shoulder_joint">
+      <command_interface name="position"/>
+      <state_interface name="position">
+        <param name="initial_value">-0.45</param>
+      </state_interface>
+      <state_interface name="velocity"/>
     </joint>
-    <joint name='joint_2' type='revolute'>
-      <pose relative_to='joint_1'>0.75 0.0 0.0 0 0 0</pose>
-      <parent link="upper_arm_link"/>
-      <child link="arm_rgbd_camera_frame"/>
-      <axis>
-        <xyz>1 0 0</xyz>
-      </axis>
-      <limit effort="500" velocity="0.15" lower="-1.570796" upper="1.5707896"/>
+    <joint name="arm_elbow_joint">
+      <command_interface name="position"/>
+      <state_interface name="position">
+        <param name="initial_value">2.8</param>
+      </state_interface>
+      <state_interface name="velocity"/>
     </joint>
-    <!-- Controller -->
-    <plugin
-      filename="ignition-gazebo-joint-position-controller-system"
-      name="ignition::gazebo::systems::JointPositionController">
-      <joint_name>joint_0</joint_name>
-      <topic>/arm/joint_0</topic>
-      <use_velocity_commands>true</use_velocity_commands>
-      <initial_position>0.5</initial_position>
-    </plugin>
-    <plugin
-      filename="ignition-gazebo-joint-position-controller-system"
-      name="ignition::gazebo::systems::JointPositionController">
-      <joint_name>joint_1</joint_name>
-      <topic>/arm/joint_1</topic>
-      <use_velocity_commands>true</use_velocity_commands>
-    </plugin>
-    <plugin
-      filename="ignition-gazebo-joint-position-controller-system"
-      name="ignition::gazebo::systems::JointPositionController">
-      <joint_name>joint_2</joint_name>
-      <topic>/arm/joint_2</topic>
-      <use_velocity_commands>true</use_velocity_commands>
-    </plugin>
-    <!-- Joint state publisher -->
-    <plugin filename="libignition-gazebo-joint-state-publisher-system.so" name="ignition::gazebo::systems::JointStatePublisher">
-      <joint_name>joint_0</joint_name>
-      <joint_name>joint_1</joint_name>
-      <joint_name>joint_2</joint_name>
-    </plugin>
-    <frame name="arm_mount_point"/>
+    <joint name="arm_wrist_joint">
+      <command_interface name="position"/>
+      <state_interface name="position">
+        <param name="initial_value">-0.8</param>
+      </state_interface>
+      <state_interface name="velocity"/>
+    </joint>
+  </ros2_control>
   </xacro:macro>
 </robot>

File: urdf/arm/arm_demo2.urdf.xacro (robot description, xacro)
@@ -10,5 +10,5 @@
   </joint>
   <link name='arm_base_link'>
-      <xacro:inertial_cylinder mass="0.17" radius="0.05" length="0.02"/>
+      <xacro:inertial_cylinder mass="0.01" radius="0.05" length="0.02"/>
       <collision name="arm_base_link_collision">
         <pose>0 0 0 0 0 0</pose>
@@ -27,7 +27,14 @@
       </visual>
     </link>
+    <joint name='joint_0' type='revolute'>
+      <origin xyz="0.25 0 0.1" rpy="0 ${M_PI/2} 0"/>
+      <parent link="arm_base_link"/>
+      <child link="lower_arm_link"/>
+      <axis xyz="0 0 1"/>
+      <limit effort="500" velocity="10" lower="-${M_PI}" upper="${M_PI}"/>
+    </joint>
     <link name='lower_arm_link'>
      <!-- <pose relative_to='arm_base_link'>0.375 0.0 0.0 0 1.570796 0</pose>-->
-    <xacro:inertial_cylinder mass="0.17" radius="0.01" length="0.5"/>
+    <xacro:inertial_cylinder mass="0.01" radius="0.01" length="0.5"/>
       <collision name='lower_link_collision'>
       <pose>0 0 0 0 0 0</pose>
@@ -49,11 +56,4 @@
       <pose relative_to='joint_2'>0.0 0 0 0 0 0</pose>
     </frame>-->
-    <joint name='joint_0' type='revolute'>
-      <origin xyz="0.25 0 0.1" rpy="0 ${M_PI/2} 0"/>
-      <parent link="arm_base_link"/>
-      <child link="lower_arm_link"/>
-      <axis xyz="0 0 1"/>
-      <limit effort="500" velocity="10" lower="-${M_PI}" upper="${M_PI}"/>
-    </joint>
 <!--
   <joint name="joint_0" type="fixed">
@@ -63,7 +63,9 @@
   </joint>
 -->
+<!--
   <gazebo reference="arm_base_joint">
     <preserveFixedJoint>true</preserveFixedJoint>
   </gazebo>
+-->
   <ros2_control name="arm_controller_hw" type="system">
     <hardware>

File: urdf/sensors/oakd.urdf.xacro (robot description, xacro)
@@ -3,5 +3,5 @@
 <xacro:macro name="oakd" params="name:=oakd parent_link *origin model:=pro">
   <xacro:include filename="$(find irobot_create_description)/urdf/common_properties.urdf.xacro"/>
-  <xacro:property name="mass"       value="0.061"/>
+  <xacro:property name="mass"       value="0.001"/>
   <xacro:property name="baseline" value="0.075" />
   <xacro:property name="M_PI"     value="3.1415926535897931" />
@@ -25,10 +25,10 @@
       </geometry>
     </visual>
-    <collision>
+   <!-- <collision>
       <origin xyz="${collision_offset_x} ${collision_offset_y} ${collision_offset_z}"/>
       <geometry>
         <box size="${collision_length_x} ${collision_length_y} ${collision_length_z}"/>
       </geometry>
-    </collision>
+    </collision>-->
     <inertial>
       <mass value="${mass}"/>

File: urdf/standard/turtlebot4.urdf.xacro (robot description, xacro)
@@ -9,5 +9,5 @@
   <xacro:include filename="$(find dis_tutorial7)/urdf/standard/tower_sensor_plate.urdf.xacro" />
   <xacro:include filename="$(find dis_tutorial7)/urdf/standard/weight_block.urdf.xacro" />
-  <xacro:include filename="$(find dis_tutorial7)/urdf/arm/arm_demo2.urdf.xacro" />
+  <xacro:include filename="$(find dis_tutorial7)/urdf/arm/arm.urdf.xacro" />
   <!-- Mechanical properties -->
   <xacro:property name="shell_z_offset"                value="${3*cm2m}" />
@@ -102,11 +102,11 @@
     <origin xyz="${oakd_pro_x_offset} ${oakd_pro_y_offset} ${oakd_pro_z_offset}"/>
   </xacro:oakd>
-  <xacro:oakd name="top_camera" model="pro" parent_link="oakd_camera_bracket">
-    <origin xyz="0.35 0 0.35" rpy="0 ${pi/2} 0"/>
-  </xacro:oakd>
-  <xacro:simple_arm parent_link="shell_link">
-    <origin xyz="0 0 1"
+  <xacro:simple_arm parent_link="tower_sensor_plate">
+    <origin xyz="0 0 0.01"
             rpy="0 0 0"/>
   </xacro:simple_arm>
+  <xacro:oakd name="top_camera" model="pro" parent_link="arm_wrist_link">
+    <origin xyz="0 0 0.065" rpy="0 -${pi/2} 0"/>
+  </xacro:oakd>
     <gazebo>
       <plugin filename="libign_ros2_control-system.so" name="ign_ros2_control::IgnitionROS2ControlPlugin">
