Commit message: temporary idiotic solution

File: urdf/sensors/oakd.urdf.xacro (robot description, xacro)
@@ -22,5 +22,5 @@
     <visual>
       <geometry>
-        <mesh filename="package://turtlebot4_description/meshes/${name}_${model}.dae" scale="1 1 1" />
+        <mesh filename="package://turtlebot4_description/meshes/oakd_${model}.dae" scale="1 1 1" />
       </geometry>
     </visual>

File: urdf/standard/turtlebot4.urdf.xacro (robot description, xacro)
@@ -3,11 +3,11 @@
   <!-- Base create3 model -->
   <xacro:include filename="$(find irobot_create_description)/urdf/create3.urdf.xacro" />
-  <xacro:include filename="$(find turtlebot4_description)/urdf/sensors/rplidar.urdf.xacro" />
-  <xacro:include filename="$(find turtlebot4_description)/urdf/sensors/oakd.urdf.xacro" />
-  <xacro:include filename="$(find turtlebot4_description)/urdf/sensors/camera_bracket.urdf.xacro" />
-  <xacro:include filename="$(find turtlebot4_description)/urdf/standard/tower_standoff.urdf.xacro" />
-  <xacro:include filename="$(find turtlebot4_description)/urdf/standard/tower_sensor_plate.urdf.xacro" />
-  <xacro:include filename="$(find turtlebot4_description)/urdf/standard/weight_block.urdf.xacro" />
-  <xacro:include filename="$(find dis_tutorial7)/urdf/arm/arm.urdf.xacro" />
+  <xacro:include filename="$(find dis_tutorial7)/urdf/sensors/rplidar.urdf.xacro" />
+  <xacro:include filename="$(find dis_tutorial7)/urdf/sensors/oakd.urdf.xacro" />
+  <xacro:include filename="$(find dis_tutorial7)/urdf/sensors/camera_bracket.urdf.xacro" />
+  <xacro:include filename="$(find dis_tutorial7)/urdf/standard/tower_standoff.urdf.xacro" />
+  <xacro:include filename="$(find dis_tutorial7)/urdf/standard/tower_sensor_plate.urdf.xacro" />
+  <xacro:include filename="$(find dis_tutorial7)/urdf/standard/weight_block.urdf.xacro" />
+  <xacro:include filename="$(find dis_tutorial7)/urdf/arm/arm_demo.urdf.xacro" />
   <!-- Mechanical properties -->
   <xacro:property name="shell_z_offset"                value="${3*cm2m}" />
@@ -102,7 +102,13 @@
     <origin xyz="${oakd_pro_x_offset} ${oakd_pro_y_offset} ${oakd_pro_z_offset}"/>
   </xacro:oakd>
+  <xacro:oakd name="top_camera" model="pro" parent_link="oakd_camera_bracket">
+    <origin xyz="0.35 0 0.35" rpy="0 ${pi/2} 0"/>
+  </xacro:oakd>
+ <!--  -->
+<!--
   <xacro:simple_arm parent_link="shell_link">
-    <origin xyz="0 0 0.5"
-            rpy="0 0 ${pi/2}"/>
+    <origin xyz="0 0 1."
+            rpy="0 0 0"/>
   </xacro:simple_arm>
+ -->
 </robot>

Commit message: fixed pointcloud rotation

File: urdf/sensors/oakd.urdf.xacro (robot description, xacro)
@@ -50,5 +50,5 @@
   </link>
   <joint name="${name}_rgb_camera_optical_joint" type="fixed">
-      <origin xyz="0 0 0" rpy="-${M_PI/2} 0.0 -${M_PI/2}"/>
+      <origin xyz="0 0 0" rpy="-0.0 0.0 -0.0"/>
       <parent link="${name}_rgb_camera_frame"/>
       <child link="${name}_rgb_camera_optical_frame"/>

File: urdf/sensors/top_camera.urdf.xacro (robot description, xacro)
@@ -50,5 +50,5 @@
   </link>
   <joint name="${name}_rgb_camera_optical_joint" type="fixed">
-      <origin xyz="0 0 0" rpy="-${M_PI/2} 0.0 -${M_PI/2}"/>
+      <origin xyz="0 0 0" rpy="-0.0 0.0 -0.0"/>
       <parent link="${name}_rgb_camera_frame"/>
       <child link="${name}_rgb_camera_optical_frame"/>
